File: Eagle/haptic_glove/haptic_glove.sch (EAGLE design)
At the start: 40 parts, among them U1 DRV2605L, U2 DRV2605L, U3 DRV2605L, U4 DRV2605L, U5 MPU-6050-1, X1 TSW-121-07-G-S, X2 TSW-121-07-G-S

Commit message: Board schematic
Parts:
- added C13, C14: 10uF, SparkFun-Capacitors:10UF-0603-6.3V-20%
- added D1: RED, SparkFun-LED:LED-RED0603
- added D2: GREEN, SparkFun-LED:LED-GREEN0603
- added D3: Yellow, SparkFun-LED:LED-YELLOW0603
- added J1: (no value), SparkFun-Connectors:JST_2MM_MALE
- added J3: (no value), SparkFun-Connectors:CONN_021X02_NO_SILK
- added R11, R12, R13: 1.5k, SparkFun-Resistors:1.5KOHM-0603-1/10W-1%
- added R14: 1k, SparkFun-Resistors:1KOHM-0603-1/10W-1%
- added R15: THERM, SparkFun-Resistors:RESISTORAXIAL-0.3
- added R16: 10k, SparkFun-Resistors:10KOHM-0603-1/10W-1%
- added R17: PROG, SparkFun-Resistors:RESISTORAXIAL-0.3
- added S1: TL32PO, switch:TL32PO
- added U6: MCP73833, SparkFun-IC-Power:MCP73833
- added X3, X4: TSW-121-07-G-S, con-samtec:TSW-121-07-G-S
Connections:
- removed net AUX_SCL: U5.AUX_CL
- removed net AUX_SDA: U5.AUX_DA
- new net N$39: X2-9.1, X3-9.1
- new net N$40: X2-10.1, X3-10.1
- new net N$41: X2-11.1, X3-11.1
- new net N$42: X2-12.1, X3-12.1
- new net N$43: X2-13.1, X3-13.1
- new net N$44: X2-14.1, X3-14.1
- new net N$45: X2-15.1, X3-15.1
- new net N$46: X2-16.1, X3-16.1
- new net N$47: X2-17.1, X3-17.1
- new net N$48: X2-18.1, X3-18.1
- new net N$49: X2-19.1, X3-19.1
- new net N$50: X2-20.1, X3-20.1
- new net N$51: C14.1, J1.+, J3.1, S1.P, U6.VBAT
- new net N$52: X1-10.1, X4-10.1
- new net N$53: X1-9.1, X4-9.1
- new net N$54: X1-8.1, X4-8.1
- new net N$55: X1-7.1, X4-7.1
- new net N$56: X1-6.1, X4-6.1
- new net N$57: X1-5.1, X4-5.1
- new net N$58: X1-4.1, X4-4.1
- new net N$59: X1-3.1, X4-3.1
- new net N$60: C13.1, D1.A, D2.A, D3.A, U6.VDD, X1-2.1, X4-2.1
- new net N$61: D1.C, R13.1
- new net N$62: D2.C, R12.1
- new net N$63: D3.C, R11.1
- new net PG: R13.2, U6.!PG
- new net PROG: R14.2, R17.2, U6.PROG
- new net STAT1: R11.2, U6.STAT1
- new net STAT2: R12.2, U6.STAT2
- new net THERM: R15.2, R16.2, U6.THERM
- net GND: now also C13.2, C14.2, J1.-, J3.2, R14.1, R15.1, R16.1, R17.1, S1.S, U6.VSS, X1-1.1, X2-21.1, X3-21.1, X4-1.1
- net N$1: now also X2-1.1, X3-1.1; no longer R2.1, U1.SDA
- net N$11: now also X1-14.1, X4-14.1
- net N$12: now also X1-18.1, X4-18.1
- net N$17: now also X2-3.1, X3-3.1; no longer R4.1, U2.SDA
- net N$18: now also X2-4.1, X3-4.1; no longer R3.1, U2.SCL
- net N$2: now also X2-2.1, X3-2.1; no longer R1.1, U1.SCL
- net N$20: now also X1-15.1, X4-15.1
- net N$21: now also X1-19.1, X4-19.1
- net N$26: now also X2-5.1, X3-5.1; no longer R6.1, U3.SDA
- net N$27: now also X2-6.1, X3-6.1; no longer R5.1, U3.SCL
- net N$29: now also X1-16.1, X4-16.1
- net N$30: now also X1-20.1, X4-20.1
- net N$35: now also X2-7.1, X3-7.1; no longer R8.1, U4.SDA
- net N$36: now also X2-8.1, X3-8.1; no longer R7.1, U4.SCL
- net N$4: now also X1-13.1, X4-13.1
- net N$5: now also X1-17.1, X4-17.1
- net SCL: now also R1.1, R3.1, R5.1, R7.1, U1.SCL, U2.SCL, U3.SCL, U4.SCL, X1-11.1, X4-11.1
- net SDA: now also R2.1, R4.1, R6.1, R8.1, U1.SDA, U2.SDA, U3.SDA, U4.SDA, X1-12.1, X4-12.1
- net VCC: now also S1.O, X1-21.1, X4-21.1
Other:
- note added: "VDD: 3.75 - 6V"
