File: Eagle/haptic_glove/haptic_glove_0_1.brd (EAGLE design)
At the start: 81 x 44.4 mm, 42 parts, among them U1 DRV2605L, U2 DRV2605L, U3 DRV2605L, U4 DRV2605L, U5 MPU-6050-1, U6 MCP73833, X1 TSW-121-07-G-S, X2 TSW-121-07-G-S, X3 TSW-121-07-G-S, X4 TSW-121-07-G-S

Commit message: Updated board design
Routing:
- net N$5: track 56.8 -> 42.4 mm
- net N$29: track 62.2 -> 60.4 mm
- net SCL: track 88.5 -> 90.2 mm
- net VCC: track 231.7 -> 233.3 mm
- net N$30: track 65.7 -> 66.5 mm
Changed lines of the file:
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@@
 <vertex x="20.32" y="16.51"/>
 </polygon>
-<wire x1="36.41" y1="44.45" x2="37.68" y2="43.18" width="0.1524" layer="1"/>
-<wire x1="37.68" y1="43.18" x2="38.1" y2="43.18" width="0.1524" layer="1"/>
-<via x="38.1" y="43.18" extent="1-16" drill="0.35"/>
-<wire x1="38.1" y1="43.18" x2="38.1" y2="41.91" width="0.1524" layer="16"/>
 <wire x1="29.63" y1="35.56" x2="27.94" y2="35.56" width="0.1524" layer="1"/>
 <via x="27.94" y="35.56" extent="1-16" drill="0.35"/>
@@
 <wire x1="81.28" y1="31.75" x2="81.28" y2="34.29" width="0.1524" layer="1"/>
 <wire x1="24.892" y1="41.91" x2="22.86" y2="41.91" width="0.1524" layer="1"/>
+<wire x1="36.41" y1="44.45" x2="37.68" y2="43.18" width="0.1524" layer="1"/>
+<wire x1="37.68" y1="43.18" x2="38.1" y2="43.18" width="0.1524" layer="1"/>
+<via x="38.1" y="43.18" extent="1-16" drill="0.35"/>
+<wire x1="38.1" y1="43.18" x2="38.1" y2="41.91" width="0.1524" layer="16"/>
 <wire x1="24.892" y1="41.91" x2="24.6888" y2="41.91" width="0" layer="19" extent="1-1"/>
 </signal>
@@
 <wire x1="54.9014" y1="58.1286" x2="54.9014" y2="53.6314" width="0.1524" layer="1"/>
 <wire x1="83.82" y1="58.1286" x2="54.9014" y2="58.1286" width="0.1524" layer="1"/>
-<wire x1="54.61" y1="49.41605" x2="53.396975" y2="48.203025" width="0.1524" layer="16"/>
-<wire x1="53.396975" y1="48.203025" x2="50.91395" y2="45.72" width="0.1524" layer="16"/>
+<wire x1="54.61" y1="49.41605" x2="50.91395" y2="45.72" width="0.1524" layer="16"/>
 <wire x1="50.91395" y1="45.72" x2="50.8" y2="45.72" width="0.1524" layer="16"/>
 <wire x1="54.61" y1="53.34" x2="54.61" y2="49.41605" width="0.1524" layer="16"/>
@@
 <wire x1="45.72" y1="46.99" x2="42.4296125" y2="46.99" width="0.1524" layer="16"/>
 <wire x1="45.72" y1="46.99" x2="46.99" y2="45.72" width="0.1524" layer="16"/>
-<wire x1="53.396975" y1="48.203025" x2="59.8988" y2="41.7012" width="0.1524" layer="16"/>
+<wire x1="55.88" y1="45.72" x2="59.8988" y2="41.7012" width="0.1524" layer="16"/>
 <wire x1="59.8988" y1="41.7012" x2="59.9097875" y2="41.7012" width="0.1524" layer="16"/>
 <wire x1="59.9097875" y1="41.7012" x2="63.5" y2="38.1109875" width="0.1524" layer="16"/>
@@
 <wire x1="92.71" y1="53.34" x2="88.6086" y2="53.34" width="0.1524" layer="1"/>
 <wire x1="88.6086" y1="53.34" x2="83.82" y2="58.1286" width="0.1524" layer="1"/>
+<wire x1="50.8" y1="45.72" x2="55.88" y2="45.72" width="0.1524" layer="16"/>
 </signal>
 <signal name="N$3">
@@
 <wire x1="59.69" y1="48.26" x2="59.69" y2="54.61" width="0.1524" layer="1"/>
 <via x="59.69" y="54.61" extent="1-16" drill="0.35"/>
-<wire x1="59.69" y1="54.61" x2="58.1286" y2="56.1714" width="0.1524" layer="16"/>
+<wire x1="59.69" y1="54.61" x2="59.3986" y2="54.9014" width="0.1524" layer="16"/>
 <wire x1="49.41605" y1="57.15" x2="48.26" y2="57.15" width="0.1524" layer="16"/>
-<wire x1="50.39465" y1="56.1714" x2="49.41605" y2="57.15" width="0.1524" layer="16"/>
-<wire x1="58.1286" y1="56.1714" x2="50.39465" y2="56.1714" width="0.1524" layer="16"/>
+<wire x1="51.66465" y1="54.9014" x2="49.41605" y2="57.15" width="0.1524" layer="16"/>
+<wire x1="59.3986" y1="54.9014" x2="51.66465" y2="54.9014" width="0.1524" layer="16"/>
 </signal>
 <signal name="N$5">
@@
 <wire x1="55.88" y1="37.795" x2="55.88" y2="39.37" width="0.1524" layer="1"/>
 <via x="55.88" y="39.37" extent="1-16" drill="0.35"/>
-<wire x1="55.88" y1="39.37" x2="55.9290125" y2="39.37" width="0.1524" layer="16"/>
-<wire x1="59.1703875" y1="39.37" x2="61.80993125" y2="39.37" width="0.1524" layer="16"/>
-<wire x1="55.9290125" y1="39.37" x2="56.4596125" y2="38.8394" width="0.1524" layer="16"/>
-<wire x1="58.6397875" y1="38.8394" x2="59.1703875" y2="39.37" width="0.1524" layer="16"/>
-<wire x1="56.4596125" y1="38.8394" x2="58.6397875" y2="38.8394" width="0.1524" layer="16"/>
-<wire x1="61.80993125" y1="39.37" x2="63.1952" y2="37.98473125" width="0.1524" layer="16"/>
-<wire x1="63.1952" y1="37.98473125" x2="63.1952" y2="35.56" width="0.1524" layer="16"/>
-<wire x1="63.1952" y1="35.56" x2="46.99" y2="35.56" width="0.1524" layer="16"/>
+<wire x1="55.88" y1="39.37" x2="55.5752" y2="39.0652" width="0.1524" layer="16"/>
+<wire x1="55.5752" y1="39.0652" x2="55.5752" y2="35.56" width="0.1524" layer="16"/>
+<wire x1="55.5752" y1="35.56" x2="46.99" y2="35.56" width="0.1524" layer="16"/>
 <wire x1="46.99" y1="35.56" x2="43.18" y2="39.37" width="0.1524" layer="16"/>
 <wire x1="43.18" y1="44.45" x2="43.18" y2="39.37" width="0.1524" layer="16"/>
@@
 <wire x1="74.93" y1="39.37" x2="71.8703875" y2="39.37" width="0.1524" layer="16"/>
 <wire x1="71.8703875" y1="39.37" x2="71.3397875" y2="38.8394" width="0.1524" layer="16"/>
-<wire x1="56.8586" y1="54.3817875" x2="56.0997875" y2="55.1406" width="0.1524" layer="16"/>
+<wire x1="59.3986" y1="51.8417875" x2="57.3697875" y2="53.8706" width="0.1524" layer="16"/>
 <wire x1="71.3397875" y1="38.8394" x2="67.72665" y2="38.8394" width="0.1524" layer="16"/>
-<wire x1="67.72665" y1="38.8394" x2="56.8586" y2="49.70745" width="0.1524" layer="16"/>
-<wire x1="56.8586" y1="49.70745" x2="56.8586" y2="54.3817875" width="0.1524" layer="16"/>
+<wire x1="67.72665" y1="38.8394" x2="59.3986" y2="47.16745" width="0.1524" layer="16"/>
+<wire x1="59.3986" y1="47.16745" x2="59.3986" y2="51.8417875" width="0.1524" layer="16"/>
 <wire x1="43.18" y1="57.15" x2="43.18" y2="49.53" width="0.1524" layer="1"/>
-<wire x1="45.1894" y1="55.1406" x2="43.18" y2="57.15" width="0.1524" layer="16"/>
-<wire x1="56.0997875" y1="55.1406" x2="45.1894" y2="55.1406" width="0.1524" layer="16"/>
+<wire x1="46.4594" y1="53.8706" x2="43.18" y2="57.15" width="0.1524" layer="16"/>
+<wire x1="57.3697875" y1="53.8706" x2="46.4594" y2="53.8706" width="0.1524" layer="16"/>
 </signal>
 <signal name="N$21">
@@
 <wire x1="69.41" y1="38.54" x2="68.58" y2="39.37" width="0.1524" layer="1"/>
 <via x="60.96" y="34.29" extent="1-16" drill="0.35"/>
-<wire x1="36.2994" y1="36.6102125" x2="36.2994" y2="37.0497875" width="0.1524" layer="16"/>
+<wire x1="37.5694" y1="36.6102125" x2="37.5694" y2="38.3197875" width="0.1524" layer="16"/>
 <wire x1="40.64" y1="41.3903875" x2="40.64" y2="49.53" width="0.1524" layer="16"/>
-<wire x1="36.2994" y1="37.0497875" x2="40.64" y2="41.3903875" width="0.1524" layer="16"/>
-<wire x1="60.96" y1="34.29" x2="38.6196125" y2="34.29" width="0.1524" layer="16"/>
-<wire x1="38.6196125" y1="34.29" x2="36.2994" y2="36.6102125" width="0.1524" layer="16"/>
+<wire x1="37.5694" y1="38.3197875" x2="40.64" y2="41.3903875" width="0.1524" layer="16"/>
+<wire x1="60.96" y1="34.29" x2="39.8896125" y2="34.29" width="0.1524" layer="16"/>
+<wire x1="39.8896125" y1="34.29" x2="37.5694" y2="36.6102125" width="0.1524" layer="16"/>
 <wire x1="62.23" y1="39.37" x2="60.96" y2="38.1" width="0.1524" layer="1"/>
 <wire x1="60.96" y1="38.1" x2="60.96" y2="34.29" width="0.1524" layer="1"/>
@@
 <wire x1="68.275" y1="36.83" x2="67.31" y2="36.83" width="0.1524" layer="1"/>
 <via x="67.31" y="36.83" extent="1-16" drill="0.35"/>
-<wire x1="64.0306" y1="30.2602125" x2="61.1797875" y2="27.4094" width="0.1524" layer="16"/>
+<wire x1="64.0306" y1="28.9902125" x2="62.4497875" y2="27.4094" width="0.1524" layer="16"/>
 <wire x1="35.9946" y1="44.0154" x2="30.48" y2="49.53" width="0.1524" layer="16"/>
 <wire x1="35.9946" y1="36.48395625" x2="35.9946" y2="44.0154" width="0.1524" layer="16"/>
 <wire x1="67.31" y1="36.83" x2="64.0306" y2="33.5506" width="0.1524" layer="16"/>
-<wire x1="64.0306" y1="33.5506" x2="64.0306" y2="30.2602125" width="0.1524" layer="16"/>
-<wire x1="61.1797875" y1="27.4094" x2="45.06915625" y2="27.4094" width="0.1524" layer="16"/>
+<wire x1="64.0306" y1="33.5506" x2="64.0306" y2="28.9902125" width="0.1524" layer="16"/>
+<wire x1="62.4497875" y1="27.4094" x2="45.06915625" y2="27.4094" width="0.1524" layer="16"/>
 <wire x1="45.06915625" y1="27.4094" x2="35.9946" y2="36.48395625" width="0.1524" layer="16"/>
 <wire x1="30.48" y1="57.15" x2="30.48" y2="49.53" width="0.1524" layer="1"/>
@@
 <wire x1="76.76" y1="41.35" x2="76.2" y2="41.91" width="0.1524" layer="1"/>
 <via x="54.61" y="41.1706" extent="1-16" drill="0.35"/>
-<wire x1="54.61" y1="41.1706" x2="53.7097" y2="40.2703" width="0.1524" layer="16"/>
-<wire x1="53.7097" y1="40.2703" x2="52.8094" y2="39.37" width="0.1524" layer="16"/>
+<wire x1="54.61" y1="43.18" x2="53.7097" y2="44.0803" width="0.1524" layer="16"/>
+<wire x1="54.61" y1="43.18" x2="54.61" y2="41.1706" width="0.1524" layer="16"/>
+<wire x1="54.61" y1="41.1706" x2="52.8094" y2="39.37" width="0.1524" layer="16"/>
 <wire x1="52.8094" y1="39.37" x2="52.07" y2="39.37" width="0.1524" layer="16"/>
 <via x="52.07" y="39.37" extent="1-16" drill="0.35"/>
@@
 <wire x1="54.61" y1="41.1706" x2="54.61" y2="41.91" width="0.1524" layer="1"/>
 <wire x1="54.61" y1="41.91" x2="59.69" y2="41.91" width="0.1524" layer="1"/>
-<wire x1="53.7097" y1="40.2703" x2="49.8997" y2="40.2703" width="0.1524" layer="16"/>
-<wire x1="49.8997" y1="40.2703" x2="44.45" y2="45.72" width="0.1524" layer="16"/>
+<wire x1="53.7097" y1="44.0803" x2="47.3597" y2="44.0803" width="0.1524" layer="16"/>
+<wire x1="47.3597" y1="44.0803" x2="45.72" y2="45.72" width="0.1524" layer="16"/>
+<wire x1="45.72" y1="45.72" x2="44.45" y2="45.72" width="0.1524" layer="16"/>
 <via x="44.45" y="45.72" extent="1-16" drill="0.35"/>
 <wire x1="44.45" y1="45.72" x2="30.48" y2="45.72" width="0.1524" layer="1"/>
@@
 <wire x1="86.36" y1="37.25" x2="85.94" y2="36.83" width="0.1524" layer="1"/>
 <via x="86.36" y="39.37" extent="1-16" drill="0.35"/>
-<wire x1="86.36" y1="39.37" x2="90.17" y2="39.37" width="0.1524" layer="16"/>
-<wire x1="90.17" y1="39.37" x2="91.44" y2="40.64" width="0.1524" layer="16"/>
+<wire x1="91.44" y1="40.64" x2="87.63" y2="40.64" width="0.1524" layer="16"/>
+<wire x1="86.36" y1="39.37" x2="87.63" y2="40.64" width="0.1524" layer="16"/>
 <via x="91.44" y="40.64" extent="1-16" drill="0.35"/>
 <wire x1="90.8446875" y1="41.3136" x2="87.9064" y2="41.3136" width="0.1524" layer="1"/>
