File: Eagle/haptic_glove/haptic_glove_0_1.brd (EAGLE design)
At the start: 81 x 44.4 mm, 46 parts, among them U1 DRV2605L, U2 DRV2605L, U3 DRV2605L, U4 DRV2605L, U5 MPU-6050-1, U6 MCP73833, X1 TSW-121-07-G-S, X2 TSW-121-07-G-S, X3 TSW-121-07-G-S, X4 TSW-121-07-G-S

Commit message: Added board V1.1
Routing:
- net N$20: track 52.2 -> 51.4 mm
Changed lines of the file:
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@@
 <wire x1="37.52" y1="37.52" x2="37.52" y2="40.64" width="0.2032" layer="1"/>
 <wire x1="85.09" y1="52.07" x2="91.44" y2="52.07" width="0.2032" layer="16"/>
-<wire x1="85.09" y1="52.07" x2="80.01" y2="46.99" width="0.2032" layer="16"/>
+<wire x1="85.09" y1="52.07" x2="78.74" y2="45.72" width="0.2032" layer="16"/>
 <via x="64.77" y="45.72" extent="1-16" drill="0.35"/>
 <wire x1="78.74" y1="45.72" x2="64.77" y2="45.72" width="0.2032" layer="16"/>
@@
 <wire x1="50.80549375" y1="45.72549375" x2="58.42549375" y2="45.72549375" width="0.2032" layer="16"/>
 <wire x1="91.44" y1="52.07" x2="95.25" y2="55.88" width="0.2032" layer="16"/>
-<wire x1="80.01" y1="46.99" x2="78.74" y2="45.72" width="0.2032" layer="16"/>
 </signal>
 <signal name="N$3">
@@
 <wire x1="59.69" y1="48.26" x2="59.69" y2="54.61" width="0.1524" layer="1"/>
 <via x="59.69" y="54.61" extent="1-16" drill="0.35"/>
-<wire x1="59.69" y1="54.61" x2="58.1286" y2="56.1714" width="0.1524" layer="16"/>
+<wire x1="59.69" y1="54.61" x2="59.3986" y2="54.9014" width="0.1524" layer="16"/>
 <wire x1="49.41605" y1="57.15" x2="48.26" y2="57.15" width="0.1524" layer="16"/>
-<wire x1="50.39465" y1="56.1714" x2="49.41605" y2="57.15" width="0.1524" layer="16"/>
-<wire x1="58.1286" y1="56.1714" x2="50.39465" y2="56.1714" width="0.1524" layer="16"/>
+<wire x1="51.66465" y1="54.9014" x2="49.41605" y2="57.15" width="0.1524" layer="16"/>
+<wire x1="59.3986" y1="54.9014" x2="51.66465" y2="54.9014" width="0.1524" layer="16"/>
 </signal>
 <signal name="N$5">
@@
 <wire x1="74.93" y1="39.37" x2="71.8703875" y2="39.37" width="0.1524" layer="16"/>
 <wire x1="71.8703875" y1="39.37" x2="71.3397875" y2="38.8394" width="0.1524" layer="16"/>
-<wire x1="56.8586" y1="54.3817875" x2="56.0997875" y2="55.1406" width="0.1524" layer="16"/>
+<wire x1="56.8586" y1="50.5717875" x2="53.5597875" y2="53.8706" width="0.1524" layer="16"/>
 <wire x1="71.3397875" y1="38.8394" x2="67.72665" y2="38.8394" width="0.1524" layer="16"/>
 <wire x1="67.72665" y1="38.8394" x2="56.8586" y2="49.70745" width="0.1524" layer="16"/>
-<wire x1="56.8586" y1="49.70745" x2="56.8586" y2="54.3817875" width="0.1524" layer="16"/>
+<wire x1="56.8586" y1="49.70745" x2="56.8586" y2="50.5717875" width="0.1524" layer="16"/>
 <wire x1="43.18" y1="57.15" x2="43.18" y2="49.53" width="0.1524" layer="1"/>
-<wire x1="45.1894" y1="55.1406" x2="43.18" y2="57.15" width="0.1524" layer="16"/>
-<wire x1="56.0997875" y1="55.1406" x2="45.1894" y2="55.1406" width="0.1524" layer="16"/>
+<wire x1="43.9194" y1="53.8706" x2="43.18" y2="54.61" width="0.1524" layer="16"/>
+<wire x1="43.18" y1="54.61" x2="43.18" y2="57.15" width="0.1524" layer="16"/>
+<wire x1="53.5597875" y1="53.8706" x2="43.9194" y2="53.8706" width="0.1524" layer="16"/>
 </signal>
 <signal name="N$21">
