File: Eagle/haptic_glove/haptic_glove_0_1.sch (EAGLE design)
At the start: 42 parts, among them U1 DRV2605L, U2 DRV2605L, U3 DRV2605L, U4 DRV2605L, U5 MPU-6050-1, U6 MCP73833, X1 TSW-121-07-G-S, X2 TSW-121-07-G-S, X3 TSW-121-07-G-S, X4 TSW-121-07-G-S

Commit message: Modified board design
Parts:
- added C1, C4, C6: 1.0uF, SparkFun-Capacitors:1.0UF-16V-10%(0402)
- added C11: 0.1uF, SparkFun-Capacitors:1.0UF-16V-10%(0402)
Connections:
- net GND: now also C1.2, C11.1, C4.2, C6.2
- net VCC: now also C1.1, C11.2, C4.1, C6.1
Changed lines of the file:
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@@
 <part name="U4" library="SparkFun-PowerIC" deviceset="DRV2605L" device=""/>
 <part name="C7" library="SparkFun-Capacitors" deviceset="1.0UF-16V-10%(0402)" device="" value="1.0uF"/>
-<part name="SUPPLY15" library="SparkFun-Aesthetics" deviceset="VCC" device=""/>
 <part name="GND15" library="SparkFun-Aesthetics" deviceset="GND" device=""/>
 <part name="C8" library="SparkFun-Capacitors" deviceset="1.0UF-16V-10%(0402)" device="" value="1.0uF"/>
-<part name="GND16" library="SparkFun-Aesthetics" deviceset="GND" device=""/>
 <part name="SUPPLY16" library="SparkFun-Aesthetics" deviceset="VCC" device=""/>
 <part name="GND17" library="SparkFun" deviceset="GND" device=""/>
@@
 <part name="GND32" library="SparkFun-Aesthetics" deviceset="GND" device=""/>
 <part name="GND33" library="SparkFun-Aesthetics" deviceset="GND" device=""/>
+<part name="C1" library="SparkFun-Capacitors" deviceset="1.0UF-16V-10%(0402)" device="" value="1.0uF"/>
+<part name="C4" library="SparkFun-Capacitors" deviceset="1.0UF-16V-10%(0402)" device="" value="1.0uF"/>
+<part name="C6" library="SparkFun-Capacitors" deviceset="1.0UF-16V-10%(0402)" device="" value="1.0uF"/>
+<part name="C11" library="SparkFun-Capacitors" deviceset="1.0UF-16V-10%(0402)" device="" value="0.1uF"/>
 </parts>
 <sheets>
@@
 <attribute name="VALUE" x="550.164" y="310.261" size="1.778" layer="96"/>
 </instance>
-<instance part="SUPPLY15" gate="G$1" x="632.46" y="332.74" smashed="yes">
-<attribute name="VALUE" x="631.444" y="336.296" size="1.778" layer="96"/>
-</instance>
 <instance part="GND15" gate="1" x="594.36" y="307.34" smashed="yes">
 <attribute name="VALUE" x="591.82" y="304.8" size="1.778" layer="96"/>
@@
 <attribute name="VALUE" x="633.984" y="322.961" size="1.778" layer="96"/>
 </instance>
-<instance part="GND16" gate="1" x="632.46" y="314.96" smashed="yes">
-<attribute name="VALUE" x="629.92" y="312.42" size="1.778" layer="96"/>
-</instance>
 <instance part="SUPPLY16" gate="G$1" x="591.82" y="332.74" smashed="yes">
 <attribute name="VALUE" x="590.804" y="336.296" size="1.778" layer="96"/>
@@
 <instance part="GND33" gate="1" x="528.32" y="401.32" smashed="yes" rot="R180">
 <attribute name="VALUE" x="530.86" y="403.86" size="1.778" layer="96" rot="R180"/>
+</instance>
+<instance part="C1" gate="G$1" x="632.46" y="266.7" smashed="yes">
+<attribute name="NAME" x="633.984" y="269.621" size="1.778" layer="95"/>
+<attribute name="VALUE" x="633.984" y="264.541" size="1.778" layer="96"/>
+</instance>
+<instance part="C4" gate="G$1" x="632.46" y="205.74" smashed="yes">
+<attribute name="NAME" x="633.984" y="208.661" size="1.778" layer="95"/>
+<attribute name="VALUE" x="633.984" y="203.581" size="1.778" layer="96"/>
+</instance>
+<instance part="C6" gate="G$1" x="632.46" y="147.32" smashed="yes">
+<attribute name="NAME" x="633.984" y="150.241" size="1.778" layer="95"/>
+<attribute name="VALUE" x="633.984" y="145.161" size="1.778" layer="96"/>
+</instance>
+<instance part="C11" gate="G$1" x="515.62" y="406.4" smashed="yes" rot="R90">
+<attribute name="NAME" x="512.699" y="407.924" size="1.778" layer="95" rot="R90"/>
+<attribute name="VALUE" x="517.779" y="407.924" size="1.778" layer="96" rot="R90"/>
 </instance>
 </instances>
@@
 <pinref part="U1" gate="DRV2605" pin="GND"/>
 <wire x1="589.28" y1="149.86" x2="594.36" y2="149.86" width="0.1524" layer="91"/>
-<wire x1="594.36" y1="149.86" x2="594.36" y2="134.62" width="0.1524" layer="91"/>
+<wire x1="594.36" y1="149.86" x2="594.36" y2="139.7" width="0.1524" layer="91"/>
 <pinref part="GND1" gate="1" pin="GND"/>
+<pinref part="C6" gate="G$1" pin="2"/>
+<wire x1="594.36" y1="139.7" x2="594.36" y2="134.62" width="0.1524" layer="91"/>
+<wire x1="632.46" y1="144.78" x2="632.46" y2="139.7" width="0.1524" layer="91"/>
+<wire x1="632.46" y1="139.7" x2="594.36" y2="139.7" width="0.1524" layer="91"/>
+<junction x="594.36" y="139.7"/>
 </segment>
 <segment>
@@
 <pinref part="U2" gate="DRV2605" pin="GND"/>
 <wire x1="589.28" y1="208.28" x2="594.36" y2="208.28" width="0.1524" layer="91"/>
-<wire x1="594.36" y1="208.28" x2="594.36" y2="193.04" width="0.1524" layer="91"/>
+<wire x1="594.36" y1="208.28" x2="594.36" y2="198.12" width="0.1524" layer="91"/>
 <pinref part="GND7" gate="1" pin="GND"/>
+<pinref part="C4" gate="G$1" pin="2"/>
+<wire x1="594.36" y1="198.12" x2="594.36" y2="193.04" width="0.1524" layer="91"/>
+<wire x1="632.46" y1="203.2" x2="632.46" y2="198.12" width="0.1524" layer="91"/>
+<wire x1="632.46" y1="198.12" x2="594.36" y2="198.12" width="0.1524" layer="91"/>
+<junction x="632.46" y="203.2"/>
+<junction x="594.36" y="198.12"/>
 </segment>
 <segment>
@@
 <pinref part="U3" gate="DRV2605" pin="GND"/>
 <wire x1="589.28" y1="266.7" x2="594.36" y2="266.7" width="0.1524" layer="91"/>
-<wire x1="594.36" y1="266.7" x2="594.36" y2="251.46" width="0.1524" layer="91"/>
+<wire x1="594.36" y1="266.7" x2="594.36" y2="259.08" width="0.1524" layer="91"/>
 <pinref part="GND11" gate="1" pin="GND"/>
+<pinref part="C1" gate="G$1" pin="2"/>
+<wire x1="594.36" y1="259.08" x2="594.36" y2="251.46" width="0.1524" layer="91"/>
+<wire x1="632.46" y1="264.16" x2="632.46" y2="259.08" width="0.1524" layer="91"/>
+<wire x1="632.46" y1="259.08" x2="594.36" y2="259.08" width="0.1524" layer="91"/>
+<junction x="632.46" y="264.16"/>
+<junction x="594.36" y="259.08"/>
 </segment>
 <segment>
@@
 <pinref part="U4" gate="DRV2605" pin="GND"/>
 <wire x1="589.28" y1="325.12" x2="594.36" y2="325.12" width="0.1524" layer="91"/>
-<wire x1="594.36" y1="325.12" x2="594.36" y2="309.88" width="0.1524" layer="91"/>
+<wire x1="594.36" y1="325.12" x2="594.36" y2="317.5" width="0.1524" layer="91"/>
 <pinref part="GND15" gate="1" pin="GND"/>
-</segment>
-<segment>
 <pinref part="C8" gate="G$1" pin="2"/>
+<wire x1="594.36" y1="317.5" x2="594.36" y2="309.88" width="0.1524" layer="91"/>
 <wire x1="632.46" y1="322.58" x2="632.46" y2="317.5" width="0.1524" layer="91"/>
-<pinref part="GND16" gate="1" pin="GND"/>
+<wire x1="632.46" y1="317.5" x2="594.36" y2="317.5" width="0.1524" layer="91"/>
+<junction x="594.36" y="317.5"/>
+<junction x="632.46" y="322.58"/>
 </segment>
 <segment>
@@
 <wire x1="528.32" y1="393.7" x2="528.32" y2="398.78" width="0.1524" layer="91"/>
 <pinref part="GND33" gate="1" pin="GND"/>
+<pinref part="C11" gate="G$1" pin="1"/>
+<wire x1="528.32" y1="398.78" x2="510.54" y2="398.78" width="0.1524" layer="91"/>
+<wire x1="510.54" y1="398.78" x2="510.54" y2="406.4" width="0.1524" layer="91"/>
+<junction x="528.32" y="398.78"/>
+<junction x="510.54" y="406.4"/>
 </segment>
 </net>
@@
 <junction x="591.82" y="154.94"/>
 <pinref part="SUPPLY2" gate="G$1" pin="VCC"/>
+<pinref part="C6" gate="G$1" pin="1"/>
+<wire x1="632.46" y1="152.4" x2="632.46" y2="157.48" width="0.1524" layer="91"/>
+<wire x1="632.46" y1="157.48" x2="612.14" y2="157.48" width="0.1524" layer="91"/>
+<wire x1="612.14" y1="157.48" x2="612.14" y2="154.94" width="0.1524" layer="91"/>
+<wire x1="612.14" y1="154.94" x2="591.82" y2="154.94" width="0.1524" layer="91"/>
 </segment>
 <segment>
@@
 <junction x="591.82" y="213.36"/>
 <pinref part="SUPPLY6" gate="G$1" pin="VCC"/>
+<pinref part="C4" gate="G$1" pin="1"/>
+<wire x1="632.46" y1="210.82" x2="632.46" y2="215.9" width="0.1524" layer="91"/>
+<wire x1="632.46" y1="215.9" x2="612.14" y2="215.9" width="0.1524" layer="91"/>
+<wire x1="612.14" y1="215.9" x2="612.14" y2="213.36" width="0.1524" layer="91"/>
+<wire x1="612.14" y1="213.36" x2="591.82" y2="213.36" width="0.1524" layer="91"/>
+<junction x="632.46" y="210.82"/>
 </segment>
 <segment>
@@
 <junction x="591.82" y="271.78"/>
 <pinref part="SUPPLY12" gate="G$1" pin="VCC"/>
-</segment>
-<segment>
-<pinref part="SUPPLY15" gate="G$1" pin="VCC"/>
-<pinref part="C8" gate="G$1" pin="1"/>
-<wire x1="632.46" y1="330.2" x2="632.46" y2="332.74" width="0.1524" layer="91"/>
+<pinref part="C1" gate="G$1" pin="1"/>
+<wire x1="632.46" y1="271.78" x2="632.46" y2="276.86" width="0.1524" layer="91"/>
+<wire x1="632.46" y1="276.86" x2="612.14" y2="276.86" width="0.1524" layer="91"/>
+<wire x1="612.14" y1="276.86" x2="612.14" y2="271.78" width="0.1524" layer="91"/>
+<wire x1="612.14" y1="271.78" x2="591.82" y2="271.78" width="0.1524" layer="91"/>
+<junction x="632.46" y="271.78"/>
 </segment>
 <segment>
@@
 <junction x="591.82" y="330.2"/>
 <pinref part="SUPPLY16" gate="G$1" pin="VCC"/>
+<pinref part="C8" gate="G$1" pin="1"/>
+<wire x1="632.46" y1="330.2" x2="632.46" y2="335.28" width="0.1524" layer="91"/>
+<wire x1="632.46" y1="335.28" x2="612.14" y2="335.28" width="0.1524" layer="91"/>
+<wire x1="612.14" y1="335.28" x2="612.14" y2="330.2" width="0.1524" layer="91"/>
+<wire x1="612.14" y1="330.2" x2="591.82" y2="330.2" width="0.1524" layer="91"/>
+<junction x="632.46" y="330.2"/>
 </segment>
 <segment>
@@
 <pinref part="P+3" gate="1" pin="VCC"/>
 <pinref part="U5" gate="G$1" pin="VDD"/>
-</segment>
-<segment>
+<pinref part="C11" gate="G$1" pin="2"/>
+<wire x1="518.16" y1="406.4" x2="533.4" y2="406.4" width="0.1524" layer="91"/>
+<wire x1="533.4" y1="406.4" x2="533.4" y2="403.86" width="0.1524" layer="91"/>
+<wire x1="533.4" y1="403.86" x2="538.48" y2="403.86" width="0.1524" layer="91"/>
+<junction x="538.48" y="403.86"/>
+<junction x="518.16" y="406.4"/>
+</segment>
+<segment>

Commit message: Added supplier BOM's
Parts:
- C1, C2, C3, C4, C5, C6, C7, C8: MF (none) -> MURATA; MPN (none) -> GRM155R61E105KA12D; OC_NEWARK (none) -> 03AC2571
- C10, C11, C12, C13, C14, C9, D1, D2, D3, J1, J3, MTR1, MTR2, MTR3, MTR4, R10, R11, R12, R13, R14, R15, R16, R17, R9, S1, SJ1, SJ2, SJ3, U1, U2, U3, U4, U5, U6, X1, X2, X3, X4: OC_NEWARK (none) -> unknown
